File: MAKER/Schématique_PCB/Schématique_PCB.kicad_sch (KiCad schematic)
At the start: 3 parts, among them U1 STM32G474RETx

Commit message: PCB
Parts:
- added C1, C10, C2, C9: 1u, Capacitor_SMD:C_0805_2012Metric_Pad1.18x1.45mm_HandSolder, symbol Device:C_Small
- added C11, C12, C13, C14, C15, C16: 10n, Capacitor_SMD:C_0805_2012Metric_Pad1.18x1.45mm_HandSolder, symbol Device:C
- added C17: 10u, Capacitor_SMD:C_0805_2012Metric_Pad1.18x1.45mm_HandSolder, symbol Device:C
- added C18, C3, C4, C5, C6: 100n, Capacitor_SMD:C_0805_2012Metric_Pad1.18x1.45mm_HandSolder, symbol Device:C_Small
- added C19, C8: 10n, Capacitor_SMD:C_0805_2012Metric_Pad1.18x1.45mm_HandSolder, symbol Device:C_Small
- added C7: 4.7u, Capacitor_SMD:C_0805_2012Metric_Pad1.18x1.45mm_HandSolder, symbol Device:C_Small
- added D2: LED, LED_SMD:LED_0805_2012Metric_Pad1.15x1.40mm_HandSolder, symbol Device:LED
- added H1, H2, H3, H4: MountingHole_Pad, MountingHole:MountingHole_3.2mm_M3_DIN965_Pad, symbol Mechanical:MountingHole_Pad
- added J1: TS1, Connector_PinHeader_2.54mm:PinHeader_1x03_P2.54mm_Vertical, symbol Connector:Conn_01x03_Pin
- added J10: TS9, Connector_PinHeader_2.54mm:PinHeader_1x03_P2.54mm_Vertical, symbol Connector:Conn_01x03_Pin
- added J11, J12, J13, J14, J15, J16: Conn_01x02_Pin, Connector_PinHeader_2.54mm:PinHeader_1x02_P2.54mm_Vertical, symbol Connector:Conn_01x02_Pin
- added J17: Screen, Connector_PinSocket_2.54mm:PinSocket_1x09_P2.54mm_Vertical, symbol Connector:Conn_01x09_Pin
- added J18: SD_Card, Connector_PinSocket_2.54mm:PinSocket_1x05_P2.54mm_Vertical, symbol Connector:Conn_01x05_Pin
- added J19: Conn_ST_STDC14, Connector_IDC:IDC-Header_2x07_P2.54mm_Vertical, symbol Connector:Conn_ST_STDC14
- added J2: 3.7V, Connector_JST:JST_PH_B2B-PH-K_1x02_P2.00mm_Vertical, symbol Connector:Conn_01x02_Pin
- added J3: TS2, Connector_PinHeader_2.54mm:PinHeader_1x03_P2.54mm_Vertical, symbol Connector:Conn_01x03_Pin
- added J4: TS3, Connector_PinHeader_2.54mm:PinHeader_1x03_P2.54mm_Vertical, symbol Connector:Conn_01x03_Pin
- added J5: TS4, Connector_PinHeader_2.54mm:PinHeader_1x03_P2.54mm_Vertical, symbol Connector:Conn_01x03_Pin
- added J6: TS5, Connector_PinHeader_2.54mm:PinHeader_1x03_P2.54mm_Vertical, symbol Connector:Conn_01x03_Pin
- added J7: TS6, Connector_PinHeader_2.54mm:PinHeader_1x03_P2.54mm_Vertical, symbol Connector:Conn_01x03_Pin
- added J8: TS7, Connector_PinHeader_2.54mm:PinHeader_1x03_P2.54mm_Vertical, symbol Connector:Conn_01x03_Pin
- added J9: TS8, Connector_PinHeader_2.54mm:PinHeader_1x03_P2.54mm_Vertical, symbol Connector:Conn_01x03_Pin
- added PS1: BU33SD5WG-TR, BU33SD5WG-TR:SOT95P280X125-5N, symbol BU33SD5WG-TR:BU33SD5WG-TR
- added R10, R11: 10k, Resistor_SMD:R_0805_2012Metric_Pad1.20x1.40mm_HandSolder, symbol Device:R
- added R12, R13, R14, R15, R16, R2: 1K, Resistor_SMD:R_0805_2012Metric_Pad1.20x1.40mm_HandSolder, symbol Device:R
- added R3: 330, Resistor_SMD:R_0805_2012Metric_Pad1.20x1.40mm_HandSolder, symbol Device:R
- added R4, R5, R6, R7, R8, R9: 100, Resistor_SMD:R_0805_2012Metric_Pad1.20x1.40mm_HandSolder, symbol Device:R
- added SW1: SW_Push, Button_Switch_SMD:SW_SPST_B3U-1000P, symbol Switch:SW_Push
- D1: footprint (none) -> LED_SMD:LED_0805_2012Metric_Pad1.15x1.40mm_HandSolder
- R1: footprint (none) -> Resistor_SMD:R_0805_2012Metric_Pad1.20x1.40mm_HandSolder
- U1: value STM32G474RETx -> STM32G474RET6
Connections:
- net GND: now also D1.1 (K), U1.15 (VSS), U1.27 (VSSA), U1.31 (VSS), U1.47 (VSS), U1.63 (VSS), C1.1, C10.2, C11.2, C12.2, C13.2, C14.2, C15.2, C16.2, C17.1, C18.1, C19.1, C2.1, C3.1, C4.1, C5.1, C6.1, C7.1, C8.2, C9.2, D2.1 (K), H1.1, H2.1, H3.1, H4.1, J1.1 (Pin_1), J10.1 (Pin_1), J11.2 (Pin_2), J12.2 (Pin_2), J13.2 (Pin_2), J14.2 (Pin_2), J15.2 (Pin_2), J16.2 (Pin_2), J17.2 (Pin_2), J19.11 (GNDDetect), J19.5 (GND), J19.7 (GND), J2.2 (Pin_2), J3.1 (Pin_1), J4.1 (Pin_1), J5.1 (Pin_1), J6.1 (Pin_1), J7.1 (Pin_1), J8.1 (Pin_1), J9.1 (Pin_1), PS1.2 (GND), R11.2, SW1.2; no longer R1.2
- net at R1.1: now also U1.33 (PB11); no longer D1.1 (K)
- net at D1.2 (A): now also R1.2; no longer U1.12 (PA0)
- net +3V3: now reaches U1.1 (VBAT)
- net +3V3: now also U1.16 (VDD), U1.28 (VREF+), U1.29 (VDDA), U1.32 (VDD), U1.48 (VDD), U1.64 (VDD), C10.1, C17.2, C19.2, C2.2, C3.2, C4.2, C5.2, C6.2, C7.2, C8.1, C9.1, J1.3 (Pin_3), J10.3 (Pin_3), J17.1 (Pin_1), J19.3 (VCC), J3.3 (Pin_3), J4.3 (Pin_3), J5.3 (Pin_3), J6.3 (Pin_3), J7.3 (Pin_3), J8.3 (Pin_3), J9.3 (Pin_3), PS1.5 (VOUT), R10.1, R12.1, R13.1, R14.1, R15.1, R16.1, R2.1, R3.1
- net TSensor3: now reaches U1.10 (PC2)
- net TSensor3: now also J4.2 (Pin_2)
- net TSensor4: now reaches U1.11 (PC3)
- net TSensor4: now also J5.2 (Pin_2)
- net Retro: now reaches U1.13 (PA1)
- net Retro: now also J17.8 (Pin_8)
- net STLINK_RX: now reaches U1.14 (PA2)
- net STLINK_RX: now also J19.13 (VCP_RX)
- net STLINK_TX: now reaches U1.17 (PA3)
- net STLINK_TX: now also J19.14 (VCP_TX)
- net SCK: now reaches U1.19 (PA5)
- net SCK: now also J17.7 (Pin_7), J18.4 (Pin_4)
- net at U1.2 (PC13): now also R6.1
- net SDO (MISO): now reaches U1.20 (PA6)
- net SDO (MISO): now also J17.9 (Pin_9), J18.3 (Pin_3)
- net SDI (MOSI): now reaches U1.21 (PA7)
- net SDI (MOSI): now also J17.6 (Pin_6), J18.2 (Pin_2)
- net TSensor5: now reaches U1.22 (PC4)
- net TSensor5: now also J6.2 (Pin_2)
- net TSensor6: now reaches U1.23 (PC5)
- net TSensor6: now also J7.2 (Pin_2)
- net Reset Screen: now reaches U1.24 (PB0)
- net Reset Screen: now also J17.4 (Pin_4)
- net D/C: now reaches U1.25 (PB1)
- net D/C: now also J17.5 (Pin_5)
- net CS Screen: now reaches U1.26 (PB2)
- net CS Screen: now also J17.3 (Pin_3)
- net at U1.3 (PC14): now also R5.1
- net SD_CS: now reaches U1.30 (PB10)
- net SD_CS: now also J18.1 (Pin_1)
- net TSensor7: now reaches U1.38 (PC6)
- net TSensor7: now also J8.2 (Pin_2)
- net TSensor8: now reaches U1.39 (PC7)
- net TSensor8: now also J9.2 (Pin_2)
- net at U1.4 (PC15): now also R4.1
- net TSensor9: now reaches U1.40 (PC8)
- net TSensor9: now also J10.2 (Pin_2)
- net SWDIO: now reaches U1.49 (PA13)
- net SWDIO: now also J19.4 (JTMS/SWDIO)
- net SWCLK: now reaches U1.50 (PA14)
- net SWCLK: now also J19.6 (JCLK/SWCLK)
- net at U1.52 (PC10): now also R9.1
- net at U1.53 (PC11): now also R8.1
- net at U1.54 (PC12): now also R7.1
- net at U1.61 (PB8): now also R11.1
- net NRST: now reaches U1.7 (PG10)
- net NRST: now also C18.2, J19.12 (~{RST}), R10.2, SW1.1
- net TSensor1: now reaches U1.8 (PC0)
- net TSensor1: now also J1.2 (Pin_2)
- net TSensor2: now reaches U1.9 (PC1)
- net TSensor2: now also J3.2 (Pin_2)
- new net: D2.2 (A), R3.2
- new net LIPO1S: C1.2, J2.1 (Pin_1), PS1.1 (VIN), PS1.3 (STBY)
- new net Reed1: C11.1, J11.1 (Pin_1), R16.2, R4.2
- new net Reed2: C12.1, J12.1 (Pin_1), R15.2, R5.2
- new net Reed3: C13.1, J13.1 (Pin_1), R14.2, R6.2
- new net Reed4: C14.1, J14.1 (Pin_1), R2.2, R7.2
- new net Reed5: C15.1, J15.1 (Pin_1), R12.2, R8.2
- new net Reed6: C16.1, J16.1 (Pin_1), R13.2, R9.2
- no-connect marks 0 -> 26
Other:
- note added: "Connecteurs"
- note added: "Mounting Holes"
- company: (none) -> Ensea
- title: (none) -> MOA_EscapeBox_schematic
- moved on the sheet: D1, R1
