File: MAKER/Schématique_PCB/Schématique_PCB.kicad_pcb (KiCad board)
At the start: 2 copper layers, 60 x 60 mm, 63 parts, among them J1 TS1, J10 TS9, J11 Conn_01x02_Pin, J12 Conn_01x02_Pin, J13 Conn_01x02_Pin, J14 Conn_01x02_Pin, J15 Conn_01x02_Pin, J16 Conn_01x02_Pin, J17 Screen, J18 SD_Card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

Commit message: MAJ PCB 4 Couches
Parts:
- J19: value Conn_ST_STDC14 -> ST-LINK; footprint Connector_IDC:IDC-Header_2x07_P2.54mm_Vertical -> Connector_PinHeader_1.27mm:PinHeader_2x07_P1.27mm_Vertical_SMD
- moved C4 26.7 mm to (179.0, 123.7), turned to 180 degrees
- moved C5 24.9 mm to (173.5, 123.3), turned to 180 degrees
- moved C3 14.9 mm to (178.9, 108.8)
- moved J19 12.0 mm to (167.8, 87.1)
- moved C7 10.1 mm to (163.1, 105.2), turned to 0 degrees
- moved C6 8.07 mm to (163.0, 107.3), turned to 0 degrees
- moved R9 4.17 mm to (176.4, 103.0)
- moved C10 2.07 mm to (171.5, 126.6)
- moved C19 2.07 mm to (168.5, 126.6)
- moved C8 2.07 mm to (174.5, 126.6)
- moved C9 2.07 mm to (176.5, 126.6)
- moved R15 2.04 mm to (161.7, 130.6), turned to -90 degrees
- moved C12 1.96 mm to (163.7, 130.5), turned to 90 degrees
- moved R8 1.90 mm to (174.3, 103.0)
- moved R7 1.89 mm to (172.3, 103.0)
Routing:
- net +3V3: track 254.1 -> 80.1 mm, vias 2 -> 38
- net GND: track 46.9 -> 132.2 mm, vias 27 -> 47
- net TSensor5: track 70.0 -> 35.5 mm, vias 3 -> 1
- net D/C: track 57.5 -> 34.1 mm, vias 2 -> 1
- net Reed3: track 46.4 -> 69.2 mm, vias 1 -> 3
- net SD_CS: track 61.1 -> 43.0 mm, vias 4 -> 1
- net SDI (MOSI): track 53.8 -> 69.9 mm, vias 2 -> 1
- net Reed6: track 60.7 -> 44.7 mm, vias 1 -> 4
- net TSensor4: track 33.1 -> 47.7 mm, vias 0 -> 1
- net NRST: track 56.0 -> 68.6 mm
- net Reed5: track 41.4 -> 53.6 mm
- net TSensor3: track 35.7 -> 47.3 mm, vias 2 -> 1
- net SCK: track 49.8 -> 61.0 mm, vias 0 -> 3
- net Net-(U1-PC10): track 15.2 -> 6.15 mm
- net SDO (MISO): track 60.6 -> 69.2 mm, vias 0 -> 3
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- added copper zone on In1.Cu, net +3V3
- added copper zone on In2.Cu, net GND
- removed copper zone on B.Cu, net GND
- removed copper zone on F.Cu, net GND
Other:
- copper layers 2 -> 4
